File: Hardware/MDR_Breakout_Board/MDR_Breakout_Board.kicad_pcb (KiCad board)
At the start: 2 copper layers, 50.8 x 88.9 mm, 14 parts, among them J1 BME688, J2 Si1145, J3 ADS1115_1, J4 ADXL345, J5 ADS1115_2, J6 BLE Friend, J7 ADS1115_3

Commit message: Updated helmet code, test CSVs
Parts:
- moved J3 1.15 mm to (160.0, 123.2)
- moved J5 1.15 mm to (162.6, 141.1)
- moved J7 1.15 mm to (162.6, 135.9)
Routing:
- net +3V3: track 145.0 -> 140.9 mm
- net /SDA: track 89.0 -> 92.4 mm
- net /SCL: track 86.6 -> 85.0 mm
- net /SCK: track 44.4 -> 45.6 mm
- net /SDO: track 44.8 -> 45.4 mm
- net GND: vias 44 -> 114
Other:
- outline, holes or cut-outs redrawn
- board text added: "Akshat Sahay Max Morel Marloon Paula Gonzalez Ruchit Patel JLCJLCJLCJLC"
- board text added: "USB"
- board text removed: "Akshat Sahay Max Morel Marloon Paula Gonzales Ruchit Patel"
