File: Hardware/CDR_Board/CDR_Board.kicad_pcb (KiCad board)
At the start: 2 copper layers, 0 parts

Commit message: CDR Board Component Placement
Component placement on 50 mil grid.
Parts:
- added C201: 1u, Capacitor_SMD:C_0805_2012Metric_Pad1.18x1.45mm_HandSolder, F.Cu at (157.5, 100.3)
- added C202: 1u, Capacitor_SMD:C_0805_2012Metric_Pad1.18x1.45mm_HandSolder, F.Cu at (165.1, 100.3)
- added C301: 1u, Capacitor_SMD:C_0805_2012Metric_Pad1.18x1.45mm_HandSolder, F.Cu at (125.7, 104.1)
- added C302: 1u, Capacitor_SMD:C_0805_2012Metric_Pad1.18x1.45mm_HandSolder, F.Cu at (133.3, 104.1)
- added C401: 100n, Capacitor_SMD:C_0805_2012Metric_Pad1.18x1.45mm_HandSolder, F.Cu at (149.9, 78.7)
- added C402: 100n, Capacitor_SMD:C_0805_2012Metric_Pad1.18x1.45mm_HandSolder, F.Cu at (157.5, 94.0)
- added C403: 1u, Capacitor_SMD:C_0805_2012Metric_Pad1.18x1.45mm_HandSolder, F.Cu at (149.9, 94.0)
- added C404: 1u, Capacitor_SMD:C_0805_2012Metric_Pad1.18x1.45mm_HandSolder, F.Cu at (146.1, 94.0)
- added C405: 100n, Capacitor_SMD:C_0805_2012Metric_Pad1.18x1.45mm_HandSolder, F.Cu at (153.7, 94.0)
- added C406: 100n, Capacitor_SMD:C_0805_2012Metric_Pad1.18x1.45mm_HandSolder, F.Cu at (153.7, 78.7)
- added C407: 100n, Capacitor_SMD:C_0805_2012Metric_Pad1.18x1.45mm_HandSolder, F.Cu at (144.8, 88.9)
- added C408: 100n, Capacitor_SMD:C_0805_2012Metric_Pad1.18x1.45mm_HandSolder, F.Cu at (144.8, 85.1)
- added C409: 100n, Capacitor_SMD:C_0805_2012Metric_Pad1.18x1.45mm_HandSolder, F.Cu at (160.0, 85.1)
- added C410: 100n, Capacitor_SMD:C_0805_2012Metric_Pad1.18x1.45mm_HandSolder, F.Cu at (160.0, 88.9)
- added C411: 100n, Capacitor_SMD:C_0805_2012Metric_Pad1.18x1.45mm_HandSolder, F.Cu at (142.2, 94.0)
- added C501: C, Capacitor_SMD:C_0805_2012Metric_Pad1.18x1.45mm_HandSolder, F.Cu at (166.4, 81.3)
- added C502: 27p, Capacitor_SMD:C_0805_2012Metric_Pad1.18x1.45mm_HandSolder, F.Cu at (134.6, 81.3)
- added C503: 27p, Capacitor_SMD:C_0805_2012Metric_Pad1.18x1.45mm_HandSolder, F.Cu at (134.6, 86.4)
- added C701: 1u, Capacitor_SMD:C_0805_2012Metric_Pad1.18x1.45mm_HandSolder, F.Cu at (125.7, 91.4)
- added C702: 0.1u, Capacitor_SMD:C_0805_2012Metric_Pad1.18x1.45mm_HandSolder, F.Cu at (125.7, 86.4)
- added D101: SMB ≥20V ≥1A, Diode_SMD:D_SOD-323_HandSoldering, F.Cu at (165.1, 105.4)
- added D301: LED, LED_SMD:LED_0805_2012Metric_Pad1.15x1.40mm_HandSolder, F.Cu at (142.2, 104.1)
- added H1: Hole, MountingHole:MountingHole_2.2mm_M2_DIN965_Pad, F.Cu at (124.5, 78.7)
- added H2: Hole, MountingHole:MountingHole_2.2mm_M2_DIN965_Pad, F.Cu at (180.3, 78.7)
- added H3: Hole, MountingHole:MountingHole_2.2mm_M2_DIN965_Pad, F.Cu at (124.5, 114.3)
- added H4: Hole, MountingHole:MountingHole_2.2mm_M2_DIN965_Pad, F.Cu at (180.3, 114.3)
- added J1: BLE Friend, Connector_PinSocket_2.54mm:PinSocket_1x09_P2.54mm_Vertical, F.Cu at (180.3, 86.4)
- added J2: nRF24L01, Connector_PinSocket_2.54mm:PinSocket_2x04_P2.54mm_Vertical, F.Cu at (172.7, 86.4)
- added J3: Battery, Connector_JST:JST_PH_S2B-PH-SM4-TB_1x02-1MP_P2.00mm_Horizontal, F.Cu at (137.2, 111.8)
- added J5: USB_C_Receptacle_USB2.0, Connector_USB:USB_C_Receptacle_Palconn_UTC16-G, F.Cu at (152.4, 113.0)
- added Q1: DMP2045U, Package_TO_SOT_SMD:SOT-23, F.Cu at (161.3, 105.4)
- added R101: 10k, Resistor_SMD:R_0805_2012Metric_Pad1.20x1.40mm_HandSolder, F.Cu at (161.3, 109.2)
- added R201: 10k, Resistor_SMD:R_0805_2012Metric_Pad1.20x1.40mm_HandSolder, F.Cu at (157.5, 105.4)
- added R301: R, Resistor_SMD:R_0805_2012Metric_Pad1.20x1.40mm_HandSolder, F.Cu at (129.5, 100.3)
- added R302: 10k, Resistor_SMD:R_0805_2012Metric_Pad1.20x1.40mm_HandSolder, F.Cu at (129.5, 108.0)
- added R303: R, Resistor_SMD:R_0805_2012Metric_Pad1.20x1.40mm_HandSolder, F.Cu at (129.5, 111.8)
- added R304: R, Resistor_SMD:R_0805_2012Metric_Pad1.20x1.40mm_HandSolder, F.Cu at (125.7, 109.2)
- added R305: 330, Resistor_SMD:R_0805_2012Metric_Pad1.20x1.40mm_HandSolder, F.Cu at (138.4, 104.1)
- added R401: 5K1, Resistor_SMD:R_0805_2012Metric_Pad1.20x1.40mm_HandSolder, F.Cu at (152.4, 100.3)
- added R402: 5K1, Resistor_SMD:R_0805_2012Metric_Pad1.20x1.40mm_HandSolder, F.Cu at (148.6, 100.3)
- added R403: 10k, Resistor_SMD:R_0805_2012Metric_Pad1.20x1.40mm_HandSolder, F.Cu at (137.2, 92.7)
- added R404: 10k, Resistor_SMD:R_0805_2012Metric_Pad1.20x1.40mm_HandSolder, F.Cu at (137.2, 96.5)
- added R501: 1k, Resistor_SMD:R_0805_2012Metric_Pad1.20x1.40mm_HandSolder, F.Cu at (144.8, 81.3)
- added R502: 10K, Resistor_SMD:R_0805_2012Metric_Pad1.20x1.40mm_HandSolder, F.Cu at (175.3, 113.0)
- added R503: 10K, Resistor_SMD:R_0805_2012Metric_Pad1.20x1.40mm_HandSolder, F.Cu at (170.2, 113.0)
- added R601: 5K1, Resistor_SMD:R_0805_2012Metric_Pad1.20x1.40mm_HandSolder, F.Cu at (164.5, 114.3)
- added R602: 5K1, Resistor_SMD:R_0805_2012Metric_Pad1.20x1.40mm_HandSolder, F.Cu at (160.7, 114.3)
- added SW1: BOOTSEL, Button_Switch_SMD:SW_Push_1P1T_NO_CK_KMR2, F.Cu at (175.3, 108.0)
- added SW2: RESET, Button_Switch_SMD:SW_Push_1P1T_NO_CK_KMR2, F.Cu at (170.2, 108.0)
- added U1: W25Q32JVSS, Package_SO:SOIC-8_5.23x5.23mm_P1.27mm, F.Cu at (166.4, 87.6)
- added U2: SOT23-5 200mA 3.3V, Package_TO_SOT_SMD:SOT-23-5, F.Cu at (161.3, 100.3)
- added U3: RP2040, Package_DFN_QFN:QFN-56-1EP_7x7mm_P0.4mm_EP3.2x3.2mm_ThermalVias, F.Cu at (152.4, 86.4)
- added U4: BQ25172, Package_SON:WSON-8-1EP_2x2mm_P0.5mm_EP0.9x1.6mm_ThermalVias, F.Cu at (129.5, 104.1)
- added U6: ADXL343, Package_LGA:LGA-14_3x5mm_P0.8mm_LayoutBorder1x6y, F.Cu at (129.5, 88.9)
- added Y1: Crystal, Crystal:Crystal_SMD_Abracon_ABM3-2Pin_5.0x3.2mm_HandSoldering, F.Cu at (139.7, 83.8)
Other:
- board outline added: 61 x 40.6 mm
